File: DE0_PSP_SCREEN.sch (KiCad schematic (older format))
At the start: 3 parts, among them P1 PSP1000LCD, P2 DE0-GPIO-0, P3 DE0-GPIO-1

Commit message: More schematic and plades headers to connect to DE0 board in pcb
Parts:
- removed P2: DE0-GPIO-0, symbol SUPP40
- removed P3: DE0-GPIO-1, symbol SUPP40
- added P?: DE0_GPIO_0, symbol CONN_20X2
- added P?: DE0_GPIO_1, symbol CONN_20X2
Connections:
- net labels added: B0, B1, B2, B3, B4, B5, B6, B7, G0, G1, G2, G3, G4, G5, G6, G7, GND, R0, R1, R2, R3, R4, R5, R6, R7
- wire segments 0 -> 58

Commit message: updated to sch
Parts:
- added C? (x2): 4.7 uF, symbol CP1
- added C? (x2): 100 n, symbol C
- added C? (x2): 10 n, symbol C
- added K?: CONN_3, symbol CONN_3
- added P4: PSP1000LED, symbol PSP1000LED
- gave numbers to parts that had none: 2
Connections:
- net GND: now also P1.39 (TEST2), P1.40 (TEST3), C?.2, C?.2, C?.2, C?.2, C?.2, C?.2, K?.3 (P3)
- net 3V3: now reaches P1.3 (VCC)
- net 3V3: now also P1.4 (VCC), P2.29 (P29), C?.1, C?.1, C?.1
- net CK: now reaches P1.30 (CK)
- net CK: now also P3.2 (P2)
- net DISP: now reaches P1.31 (DISP)
- net DISP: now also P3.3 (P3)
- net Hsync: now reaches P1.32 (Hsync)
- net Hsync: now also P3.4 (P4)
- net Vsync: now reaches P1.33 (Vsync)
- net Vsync: now also P3.5 (P5)
- net +5VA: now reaches P1.35 (AVDD)
- net +5VA: now also P1.36 (AVDD), C?.1, C?.1, C?.1, K?.2 (PM)
- net +5V: now reaches P2.11 (P11)
- net +5V: now also K?.1 (P1)
