File: DE0_PSP_SCREEN.sch (KiCad schematic (older format))
At the start: 5 parts, among them P1 PSP1000LCD, P2 DE0_GPIO_0, P3 DE0_GPIO_1, P4 PSP1000LED, P5 CONN_2

Commit message: More changes
Connections:
- wire segments 100 -> 121
Changed lines of the file:
@@
-EESchema Schematic File Version 2  date Thu 08 Nov 2012 00:17:25 CET
+EESchema Schematic File Version 2  date Thu 08 Nov 2012 11:50:00 CET
 LIBS:power
 LIBS:device
@@
 Sheet 1 4
 Title ""
-Date "7 nov 2012"
+Date "8 nov 2012"
 Rev ""
 Comp ""
@@
 Text Label 3050 2550 2    60   ~ 0
 B7
-Text Label 9250 1550 2    60   ~ 0
+Text Label 9250 5550 0    60   ~ 0
 R0
-Text Label 9250 1650 2    60   ~ 0
+Text Label 8150 5550 2    60   ~ 0
 R1
-Text Label 8150 1750 0    60   ~ 0
+Text Label 9250 5350 0    60   ~ 0
 R2
-Text Label 9250 1750 2    60   ~ 0
+Text Label 8150 5350 2    60   ~ 0
 R3
-Text Label 8150 1850 0    60   ~ 0
+Text Label 9250 5250 0    60   ~ 0
 R4
-Text Label 8150 1950 0    60   ~ 0
+Text Label 9250 5150 0    60   ~ 0
 R6
-Text Label 9250 1850 2    60   ~ 0
+Text Label 8150 5250 2    60   ~ 0
 R5
-Text Label 9250 1950 2    60   ~ 0
+Text Label 8150 5150 2    60   ~ 0
 R7
 $Comp
@@
 	1    0    0    -1
 $EndComp
-Text Label 8150 2150 0    60   ~ 0
+Text Label 9250 5050 0    60   ~ 0
 G0
-Text Label 9250 2150 2    60   ~ 0
+Text Label 8150 5050 2    60   ~ 0
 G1
-Text Label 8150 2250 0    60   ~ 0
+Text Label 9250 4950 0    60   ~ 0
 G2
-Text Label 9250 2250 2    60   ~ 0
+Text Label 8150 4950 2    60   ~ 0
 G3
-Text Label 8150 2350 0    60   ~ 0
+Text Label 9250 4850 0    60   ~ 0
 G4
-Text Label 9250 2350 2    60   ~ 0
+Text Label 8150 4850 2    60   ~ 0
 G5
-Text Label 8150 2450 0    60   ~ 0
+Text Label 9250 4750 0    60   ~ 0
 G6
-Text Label 9250 2450 2    60   ~ 0
+Text Label 8150 4750 2    60   ~ 0
 G7
-Text Label 9250 2850 2    60   ~ 0
+Text Label 9250 4250 0    60   ~ 0
 B7
-Text Label 8150 2550 0    60   ~ 0
+Text Label 8150 4650 2    60   ~ 0
 B0
-Text Label 9250 2550 2    60   ~ 0
+Text Label 9250 4650 0    60   ~ 0
 B1
-Text Label 8150 2650 0    60   ~ 0
+Text Label 8150 4550 2    60   ~ 0
 B2
-Text Label 9250 2650 2    60   ~ 0
+Text Label 9250 4450 0    60   ~ 0
 B3
-Text Label 8150 2750 0    60   ~ 0
+Text Label 8150 4450 2    60   ~ 0
 B4
-Text Label 9250 2750 2    60   ~ 0
+Text Label 9250 4350 0    60   ~ 0
 B5
-Text Label 8150 2850 0    60   ~ 0
+Text Label 8150 4350 2    60   ~ 0
 B6
 $Comp
@@
 Text Label 3050 2050 2    60   ~ 0
 Vsync
+Text Label 8150 4250 2    60   ~ 0
+CK
+Text Label 9250 4150 0    60   ~ 0
+DISP
+Text Label 8150 4150 2    60   ~ 0
+Hsync
 Text Label 9250 4050 0    60   ~ 0
-CK
-Text Label 8150 4150 2    60   ~ 0
-DISP
-Text Label 9250 4150 0    60   ~ 0
-Hsync
-Text Label 8150 4250 2    60   ~ 0
 Vsync
 $Comp
@@
 Wire Wire Line
 	2900 2550 3050 2550
-Wire Wire Line
-	9100 1550 9250 1550
 Wire Wire Line
 	9100 1650 9250 1650
@@
 Wire Wire Line
 	1750 4000 1500 4000
-Text Label 9250 4250 0    60   ~ 0
+Text Label 8100 3650 0    60   ~ 0
 dimm
 Wire Wire Line
@@
 Wire Wire Line
 	9100 4350 9250 4350
-Text Label 9250 4350 0    60   ~ 0
+Text Label 7900 3800 0    60   ~ 0
 5vENA
-Text Label 8150 4350 2    60   ~ 0
+Text Label 7650 3850 2    60   ~ 0
 3v3ENA
 Wire Wire Line
@@
 Connection ~ 9550 5000
 $Comp
-L GND #PWR06
+L GND #PWR05
 U 1 1 508D5FD4
 P 9900 5250
-F 0 "#PWR06" H 9900 5250 30  0001 C CNN
+F 0 "#PWR05" H 9900 5250 30  0001 C CNN
 F 1 "GND" H 9900 5180 30  0001 C CNN
 	1    9900 5250
@@
 6-24V
 $Comp
-L GND #PWR07
+L GND #PWR06
 U 1 1 50927877
 P 2850 5350
-F 0 "#PWR07" H 2850 5350 30  0001 C CNN
+F 0 "#PWR06" H 2850 5350 30  0001 C CNN
 F 1 "GND" H 2850 5280 30  0001 C CNN
 	1    2850 5350
@@
 Text Label 2000 6550 2    60   ~ 0
 CMD
-Text Label 8150 4450 2    60   ~ 0
+Text Label 8150 5850 2    60   ~ 0
 DAT3
-Text Label 9250 4450 0    60   ~ 0
+Text Label 9250 5750 0    60   ~ 0
 DAT2
-Text Label 8150 4550 2    60   ~ 0
+Text Label 8150 5650 2    60   ~ 0
 DAT1
-Text Label 9250 4650 0    60   ~ 0
+Text Label 8150 5750 2    60   ~ 0
 CLK
-Text Label 8150 4650 2    60   ~ 0
+Text Label 9250 5850 0    60   ~ 0
 CMD
 Wire Wire Line
@@
 Text Label 1500 4000 2    60   ~ 0
 Vout-
+Wire Wire Line
+	9100 4750 9250 4750
+Wire Wire Line
+	8300 4750 8150 4750
+Wire Wire Line
+	8300 4850 8150 4850
+Wire Wire Line
+	8300 4950 8150 4950
+Wire Wire Line
+	8300 5050 8150 5050
+Wire Wire Line
+	8300 5150 8150 5150
+Wire Wire Line
+	8300 5250 8150 5250
+Wire Wire Line
+	8300 5350 8150 5350
+Wire Wire Line
+	9100 5350 9250 5350
+Wire Wire Line
+	9100 5250 9250 5250
+Wire Wire Line
+	9100 5150 9250 5150
+Wire Wire Line
+	9100 5050 9250 5050
+Wire Wire Line
+	9100 4950 9250 4950
+Wire Wire Line
+	9100 4850 9250 4850
+Wire Wire Line
+	8300 5550 8150 5550
+Wire Wire Line
+	8300 5650 8150 5650
+Wire Wire Line
+	9100 5550 9250 5550
+Wire Wire Line
+	9100 5650 9250 5650
+Text Label 9250 5650 0    60   ~ 0
+DAT0
+Wire Wire Line
+	8300 5750 8150 5750
+Wire Wire Line
+	9100 5750 9250 5750
+Wire Wire Line
+	8300 5850 8150 5850
+Wire Wire Line
+	9100 5850 9250 5850
 $EndSCHEMATC

Commit message: Close to done
Connections:
- net labels removed: 6-24V
- wire segments 121 -> 100
Changed lines of the file:
@@
-EESchema Schematic File Version 2  date Thu 08 Nov 2012 11:50:00 CET
+EESchema Schematic File Version 2  date Sun 11 Nov 2012 16:06:29 CET
 LIBS:power
 LIBS:device
@@
 Sheet 1 4
 Title ""
-Date "8 nov 2012"
+Date "11 nov 2012"
 Rev ""
 Comp ""
@@
 Text Label 9250 4650 0    60   ~ 0
 B1
-Text Label 8150 4550 2    60   ~ 0
+Text Label 8100 3450 2    60   ~ 0
 B2
 Text Label 9250 4450 0    60   ~ 0
@@
 	2900 2550 3050 2550
 Wire Wire Line
-	9100 1650 9250 1650
-Wire Wire Line
-	9100 1750 9250 1750
-Wire Wire Line
-	8300 1750 8150 1750
-Wire Wire Line
-	8300 1850 8150 1850
-Wire Wire Line
-	9100 1850 9250 1850
-Wire Wire Line
-	9100 1950 9250 1950
-Wire Wire Line
-	8300 1950 8150 1950
-Wire Wire Line
-	8300 2150 8150 2150
-Wire Wire Line
-	8300 2250 8150 2250
-Wire Wire Line
-	8300 2350 8150 2350
-Wire Wire Line
-	8300 2450 8150 2450
-Wire Wire Line
-	9100 2150 9250 2150
-Wire Wire Line
-	9100 2250 9250 2250
-Wire Wire Line
-	9100 2350 9250 2350
-Wire Wire Line
-	9100 2450 9250 2450
-Wire Wire Line
-	8300 2550 8150 2550
-Wire Wire Line
-	8300 2650 8150 2650
-Wire Wire Line
-	8300 2750 8150 2750
-Wire Wire Line
-	8300 2850 8150 2850
-Wire Wire Line
-	9100 2550 9250 2550
-Wire Wire Line
-	9100 2650 9250 2650
-Wire Wire Line
-	9100 2750 9250 2750
-Wire Wire Line
-	9100 2850 9250 2850
-Wire Wire Line
 	9450 2950 9100 2950
 Wire Wire Line
@@
 Wire Wire Line
 	1750 4000 1500 4000
-Text Label 8100 3650 0    60   ~ 0
+Text Label 8300 2850 2    60   ~ 0
 dimm
 Wire Wire Line
@@
 F0 "Sheet508A6549" 60
 F1 "file508A6549.sch" 60
-F2 "V6-24" I L 5250 3700 60
-F3 "DE0_5v" I L 5250 3850 60
-F4 "DE0_3v3" I L 5250 4000 60
-F5 "5Vreg" I R 6550 3700 60
-F6 "3v3Vreg" I R 6550 3850 60
-F7 "5vENA" I L 5250 4250 60
-F8 "3v3ENA" I L 5250 4400 60
+F2 "DE0_5v" I L 5250 3850 60
+F3 "DE0_3v3" I L 5250 4000 60
+F4 "5Vreg" I R 6550 3700 60
+F5 "3v3Vreg" I R 6550 3850 60
+F6 "5vENA" I L 5250 4250 60
+F7 "3v3ENA" I L 5250 4400 60
+F8 "V6_24" I L 5250 3700 60
 $EndSheet
 Text Label 6550 3700 0    60   ~ 0
@@
 Wire Wire Line
 	9100 4350 9250 4350
-Text Label 7900 3800 0    60   ~ 0
+Text Label 8300 2350 2    60   ~ 0
 5vENA
-Text Label 7650 3850 2    60   ~ 0
+Text Label 9100 1550 0    60   ~ 0
 3v3ENA
 Wire Wire Line
@@
 $EndComp
 Wire Wire Line
-	3000 5150 2850 5150
-Wire Wire Line
 	3000 5350 2850 5350
-Text Label 2850 5150 2    60   ~ 0
-6-24V
 $Comp
 L GND #PWR06
@@
 	1    0    0    -1
 $EndComp
-Text Label 5250 3700 2    60   ~ 0
-6-24V
 $Sheet
 S 2000 5950 1500 1250
@@
 	9100 4450 9250 4450
 Wire Wire Line
-	8300 4550 8150 4550
-Wire Wire Line
 	9100 4650 9250 4650
 Wire Wire Line
@@
 Wire Wire Line
 	9100 5850 9250 5850
+Wire Wire Line
+	3000 5150 2800 5150
+Wire Wire Line
+	2800 5150 2800 3700
+Wire Wire Line
+	2800 3700 5250 3700
+Wire Wire Line
+	8300 3450 8100 3450
 $EndSCHEMATC
