File: file508A6549.sch (KiCad schematic (older format))
At the start: 7 parts

Commit message: Added power supply
Parts:
- added C11: 22nF, symbol C
- added C12: 100pF, symbol C
- added C13: 22uF, symbol C
- added C14: 10nF, symbol C
- added C5: 10uF, symbol C
- added D3: B230A, symbol DIODESCH
- added D4, D5: LED, symbol LED
- added K2: CONN_3, symbol CONN_3
- added L2: 3.3uH, symbol INDUCTOR_SMALL
- added R4, R7: 100k, symbol R
- added R5: 49.9k, symbol R
- added R6: 9.53, symbol R
- added R8, R9: R, symbol R
- added U2: AP5100, symbol AP5100
- added U3: LP2985, symbol LP2985
- gave numbers to parts that had none: 7
Connections:
- net labels added: 3v3ENA, 3v3Vreg, 5vENA, DE0_3v3, DE0_5v, V6-24, Vin, Vout3v3, Vout5v
- net labels removed: +5V, +5VA, 3V3
- wire segments 11 -> 51
Other:
- note added: "Jumper to select between 3v3 from \nDE0 board or reg"
- note added: "Jumper to select between 5v from \nDE0 board or step down reg"
- note added: "L = (Vout*(Vin-Vout))/(Vin*IL*fSW)\nIL = inductor ripple current\nfSW = buck converter switching frequency"
- note added: "R1 = R2*(Vout/0.81-1)"

Commit message: Started on routing power supply
Parts:
- removed C4: 10 n, symbol C
- removed C6: 100 n, symbol C
Connections:
- net 3v3Vreg: no longer C7.1
- net V6-24: now also C5.2
- net Vout3v3: now also C7.1
- net at C11.2, L2.1, U2.6 (SW): now also D3.2 (K)
Other:
- moved on the sheet: C7
Changed lines of the file:
@@
-EESchema Schematic File Version 2  date Sun 28 Oct 2012 15:35:36 CET
+EESchema Schematic File Version 2  date Mon 29 Oct 2012 16:35:26 CET
 LIBS:power
 LIBS:device
@@
 Sheet 3 3
 Title "power supply"
-Date "28 oct 2012"
+Date "29 oct 2012"
 Rev "0.1"
 Comp ""
@@
 L CP1 C7
 U 1 1 508A6583
-P 1850 1250
-F 0 "C7" H 1900 1350 50  0000 L CNN
-F 1 "4.7 uF" H 1900 1150 50  0000 L CNN
-	1    1850 1250
-	1    0    0    -1
-$EndComp
-$Comp
-L C C6
-U 1 1 508A6589
-P 1550 1250
-F 0 "C6" H 1600 1350 50  0000 L CNN
-F 1 "100 n" H 1600 1150 50  0000 L CNN
-	1    1550 1250
-	1    0    0    -1
-$EndComp
-$Comp
-L C C4
-U 1 1 508A658F
-P 1250 1250
-F 0 "C4" H 1300 1350 50  0000 L CNN
-F 1 "10 n" H 1300 1150 50  0000 L CNN
-	1    1250 1250
-	1    0    0    -1
-$EndComp
-Wire Wire Line
-	1000 1050 1850 1050
-Connection ~ 1550 1050
-Wire Wire Line
-	1250 1450 1850 1450
-Connection ~ 1550 1450
-Wire Wire Line
-	1550 1450 1550 1650
-Wire Wire Line
-	1550 1050 1550 850
-$Comp
-L GND #PWR08
-U 1 1 508A659D
-P 1550 1650
-F 0 "#PWR08" H 1550 1650 30  0001 C CNN
-F 1 "GND" H 1550 1580 30  0001 C CNN
-	1    1550 1650
-	1    0    0    -1
-$EndComp
+P 9550 3250
+F 0 "C7" H 9600 3350 50  0000 L CNN
+F 1 "4.7 uF" H 9600 3150 50  0000 L CNN
+	1    9550 3250
+	1    0    0    -1
+$EndComp
+Wire Wire Line
+	1000 1050 1000 850
 $Comp
 L CP1 C10
@@
 	2800 1050 2800 850
 $Comp
-L GND #PWR09
+L GND #PWR08
 U 1 1 508A66C1
 P 2800 1650
-F 0 "#PWR09" H 2800 1650 30  0001 C CNN
+F 0 "#PWR08" H 2800 1650 30  0001 C CNN
 F 1 "GND" H 2800 1580 30  0001 C CNN
 	1    2800 1650
@@
 	1200 2650 1200 2700
 $Comp
-L GND #PWR010
+L GND #PWR09
 U 1 1 508D28C4
 P 1200 2700
-F 0 "#PWR010" H 1200 2700 30  0001 C CNN
+F 0 "#PWR09" H 1200 2700 30  0001 C CNN
 F 1 "GND" H 1200 2630 30  0001 C CNN
 	1    1200 2700
@@
 Connection ~ 3850 4500
 $Comp
-L GND #PWR011
+L GND #PWR010
 U 1 1 508D301C
 P 3850 4700
-F 0 "#PWR011" H 3850 4700 30  0001 C CNN
+F 0 "#PWR010" H 3850 4700 30  0001 C CNN
 F 1 "GND" H 3850 4630 30  0001 C CNN
 	1    3850 4700
@@
 	7800 3300 7800 3400
 $Comp
-L GND #PWR012
+L GND #PWR011
 U 1 1 508D3C07
 P 7800 3400
-F 0 "#PWR012" H 7800 3400 30  0001 C CNN
+F 0 "#PWR011" H 7800 3400 30  0001 C CNN
 F 1 "GND" H 7800 3330 30  0001 C CNN
 	1    7800 3400
@@
 	9300 4150 9300 4250
 $Comp
-L GND #PWR013
+L GND #PWR012
 U 1 1 508D3EFA
 P 9300 4250
-F 0 "#PWR013" H 9300 4250 30  0001 C CNN
+F 0 "#PWR012" H 9300 4250 30  0001 C CNN
 F 1 "GND" H 9300 4180 30  0001 C CNN
 	1    9300 4250
@@
 Text Label 7800 1050 2    60   ~ 0
 3v3Vreg
-Text Label 1550 850  2    60   ~ 0
+Text Label 1000 850  2    60   ~ 0
 3v3Vreg
 Text Label 7800 1150 2    60   ~ 0
@@
 	1    0    0    -1
 $EndComp
-Connection ~ 1250 1050
 Wire Wire Line
 	1000 1550 1000 1650
-Wire Wire Line
-	1000 2050 1250 2050
-Wire Wire Line
-	1250 2050 1250 1450
 Wire Wire Line
 	2250 1550 2250 1650
@@
 Text Label 1000 6000 0    60   ~ 0
 5vENA
+$Comp
+L GND #PWR013
+U 1 1 508E96BB
+P 1000 2050
+F 0 "#PWR013" H 1000 2050 30  0001 C CNN
+F 1 "GND" H 1000 1980 30  0001 C CNN
+	1    1000 2050
+	1    0    0    -1
+$EndComp
+Wire Wire Line
+	9550 3450 9550 4200
+Wire Wire Line
+	9550 4200 9300 4200
+Connection ~ 9300 4200
+Connection ~ 9550 3050
+Connection ~ 1400 3050
+Connection ~ 3450 3300
+Connection ~ 3450 3700
 $EndSCHEMATC

Commit message: lots of changes
Parts:
- L2: value 3.3uH -> 3.3uH SPM6530
Connections:
- net 5vENA: now also R4.2
- net V6-24: now also R4.1
Changed lines of the file:
@@
-EESchema Schematic File Version 2  date Thu 01 Nov 2012 14:43:35 CET
+EESchema Schematic File Version 2  date Thu 08 Nov 2012 00:17:25 CET
 LIBS:power
 LIBS:device
@@
 Sheet 3 4
 Title "power supply"
-Date "1 nov 2012"
+Date "7 nov 2012"
 Rev "0.1"
 Comp ""
@@
 P 4000 3300
 F 0 "L2" H 4000 3400 50  0000 C CNN
-F 1 "3.3uH" H 4000 3250 50  0000 C CNN
+F 1 "3.3uH SPM6530" H 4000 3250 50  0000 C CNN
 	1    4000 3300
 	1    0    0    -1
@@
 Connection ~ 3450 3300
 Connection ~ 3450 3700
+Connection ~ 1750 3050
+Connection ~ 1750 3550
 $EndSCHEMATC

Commit message: Close to done
Connections:
- net V6-24 renamed V6_24
Changed lines of the file:
@@
-EESchema Schematic File Version 2  date Thu 08 Nov 2012 00:17:25 CET
+EESchema Schematic File Version 2  date Sun 11 Nov 2012 16:06:29 CET
 LIBS:power
 LIBS:device
@@
 Sheet 3 4
 Title "power supply"
-Date "7 nov 2012"
+Date "11 nov 2012"
 Rev "0.1"
 Comp ""
@@
 	2800 1050 2800 850
 $Comp
-L GND #PWR09
+L GND #PWR08
 U 1 1 508A66C1
 P 2800 1650
-F 0 "#PWR09" H 2800 1650 30  0001 C CNN
+F 0 "#PWR08" H 2800 1650 30  0001 C CNN
 F 1 "GND" H 2800 1580 30  0001 C CNN
 	1    2800 1650
@@
 	1950 3550 1250 3550
 Wire Wire Line
-	1950 3050 1250 3050
+	650  3050 1950 3050
 $Comp
 L R R4
@@
 Text Label 1250 3550 2    60   ~ 0
 5vENA
-Text Label 1250 3050 2    60   ~ 0
-Vin
 $Comp
 L C C5
@@
 	1200 2650 1200 2700
 $Comp
-L GND #PWR010
+L GND #PWR09
 U 1 1 508D28C4
 P 1200 2700
-F 0 "#PWR010" H 1200 2700 30  0001 C CNN
+F 0 "#PWR09" H 1200 2700 30  0001 C CNN
 F 1 "GND" H 1200 2630 30  0001 C CNN
 	1    1200 2700
@@
 Connection ~ 3850 4500
 $Comp
-L GND #PWR011
+L GND #PWR010
 U 1 1 508D301C
 P 3850 4700
-F 0 "#PWR011" H 3850 4700 30  0001 C CNN
+F 0 "#PWR010" H 3850 4700 30  0001 C CNN
 F 1 "GND" H 3850 4630 30  0001 C CNN
 	1    3850 4700
@@
 	7800 3300 7800 3400
 $Comp
-L GND #PWR012
+L GND #PWR011
 U 1 1 508D3C07
 P 7800 3400
-F 0 "#PWR012" H 7800 3400 30  0001 C CNN
+F 0 "#PWR011" H 7800 3400 30  0001 C CNN
 F 1 "GND" H 7800 3330 30  0001 C CNN
 	1    7800 3400
@@
 	9300 4150 9300 4250
 $Comp
-L GND #PWR013
+L GND #PWR012
 U 1 1 508D3EFA
 P 9300 4250
-F 0 "#PWR013" H 9300 4250 30  0001 C CNN
+F 0 "#PWR012" H 9300 4250 30  0001 C CNN
 F 1 "GND" H 9300 4180 30  0001 C CNN
 	1    9300 4250
@@
 Connection ~ 2500 1050
 Text HLabel 1000 4800 0    60   Input ~ 0
-V6-24
+V6_24
 Text HLabel 1000 5000 0    60   Input ~ 0
 DE0_5v
@@
 Text HLabel 1000 5600 0    60   Input ~ 0
 3v3Vreg
-Text Label 1000 4800 0    60   ~ 0
-Vin
 Text Label 1000 5000 0    60   ~ 0
 DE0_5v
@@
 5vENA
 $Comp
-L GND #PWR014
+L GND #PWR013
 U 1 1 508E96BB
 P 1000 2050
-F 0 "#PWR014" H 1000 2050 30  0001 C CNN
+F 0 "#PWR013" H 1000 2050 30  0001 C CNN
 F 1 "GND" H 1000 1980 30  0001 C CNN
 	1    1000 2050
@@
 Connection ~ 1750 3050
 Connection ~ 1750 3550
+Wire Wire Line
+	650  3050 650  4550
+Wire Wire Line
+	650  4550 1150 4550
+Wire Wire Line
+	1150 4550 1150 4800
+Wire Wire Line
+	1150 4800 1000 4800
 $EndSCHEMATC
